File: board/BatteryCurrentMonitor.sch (KiCad schematic (older format))
At the start: 3 parts, among them U4 INA260

Commit message: Rev 2 of board layout, WIP
Parts:
- C16, C17: footprint Capacitor_SMD:C_0805_2012Metric -> Capacitor_SMD:C_0805_2012Metric_Pad1.15x1.40mm_HandSolder
Changed lines of the file:
@@
 EESchema Schematic File Version 4
 LIBS:MPPTSolarCharger-cache
-EELAYER 26 0
+EELAYER 30 0
 EELAYER END
 $Descr A4 11693 8268
@@
 F 0 "C16" H 4915 3996 50  0000 L CNN
 F 1 "100nF" H 4915 3905 50  0000 L CNN
-F 2 "Capacitor_SMD:C_0805_2012Metric" H 4838 3800 50  0001 C CNN
+F 2 "Capacitor_SMD:C_0805_2012Metric_Pad1.15x1.40mm_HandSolder" H 4838 3800 50  0001 C CNN
 F 3 "~" H 4800 3950 50  0001 C CNN
 	1    4800 3950
@@
 F 0 "C17" H 6065 2896 50  0000 L CNN
 F 1 "100nF" H 6065 2805 50  0000 L CNN
-F 2 "Capacitor_SMD:C_0805_2012Metric" H 5988 2700 50  0001 C CNN
+F 2 "Capacitor_SMD:C_0805_2012Metric_Pad1.15x1.40mm_HandSolder" H 5988 2700 50  0001 C CNN
 F 3 "~" H 5950 2850 50  0001 C CNN
 	1    5950 2850
