File: board/MCU.sch (KiCad schematic (older format))
At the start: 3 parts, among them J3 Conn_01x06

Commit message: Rev 2 of board layout, WIP
Parts:
- R8, R9: footprint Resistor_SMD:R_0805_2012Metric -> Resistor_SMD:R_0805_2012Metric_Pad1.15x1.40mm_HandSolder
Changed lines of the file:
@@
 EESchema Schematic File Version 4
 LIBS:MPPTSolarCharger-cache
-EELAYER 26 0
+EELAYER 30 0
 EELAYER END
 $Descr A4 11693 8268
@@
 F 0 "R8" H 4520 2946 50  0000 L CNN
 F 1 "4.3K" H 4520 2855 50  0000 L CNN
-F 2 "Resistor_SMD:R_0805_2012Metric" V 4380 2900 50  0001 C CNN
+F 2 "Resistor_SMD:R_0805_2012Metric_Pad1.15x1.40mm_HandSolder" V 4380 2900 50  0001 C CNN
 F 3 "~" H 4450 2900 50  0001 C CNN
 	1    4450 2900
@@
 F 0 "R9" H 5070 2946 50  0000 L CNN
 F 1 "4.3K" H 5070 2855 50  0000 L CNN
-F 2 "Resistor_SMD:R_0805_2012Metric" V 4930 2900 50  0001 C CNN
+F 2 "Resistor_SMD:R_0805_2012Metric_Pad1.15x1.40mm_HandSolder" V 4930 2900 50  0001 C CNN
 F 3 "~" H 5000 2900 50  0001 C CNN
 	1    5000 2900
