File: board/PowerStage.sch (KiCad schematic (older format))
At the start: 40 parts, among them J1 Screw_Terminal_01x02, J2 Screw_Terminal_01x02, Q1 PSMN5R5-60YS, Q2 PSMN5R5-60YS, Q3 PSMN5R5-60YS, U1 LM350_TO220, U2 MIC4605-1YM

Commit message: Rev 2 of board layout, WIP
Parts:
- removed C11: 1000uF, Capacitor_THT:CP_Radial_D16.0mm_P7.50mm, symbol Device:CP
- removed JP2, JP4: Jumper_NC_Small, Connector_PinHeader_2.54mm:PinHeader_1x02_P2.54mm_Vertical, symbol Device:Jumper_NC_Small
- removed R5: 3.3, Resistor_SMD:R_0805_2012Metric, symbol Device:R
- C1, C12, C13, C2, C8, C9: footprint Capacitor_SMD:C_0805_2012Metric -> Capacitor_SMD:C_0805_2012Metric_Pad1.15x1.40mm_HandSolder
- C5, C7: footprint Capacitor_SMD:C_0805_2012Metric -> Capacitor_SMD:C_1210_3225Metric_Pad1.42x2.65mm_HandSolder
- D1, D2: footprint Diode_THT:D_DO-35_SOD27_P7.62mm_Horizontal -> Diode_SMD:D_SOD-323_HandSoldering
- J1, J2: footprint TerminalBlock_Phoenix:TerminalBlock_Phoenix_MKDS-3-2-5.08_1x02_P5.08mm_Horizontal -> Saintgimp:Phoenix_Contact_MKDS_5-2-952
- R1, R2, R3, R4, R7: footprint Resistor_SMD:R_0805_2012Metric -> Resistor_SMD:R_0805_2012Metric_Pad1.15x1.40mm_HandSolder
- R6: footprint Resistor_SMD:R_0805_2012Metric -> Resistor_SMD:R_1206_3216Metric_Pad1.42x1.75mm_HandSolder
Connections:
- wire segments 123 -> 114
Other:
- note added: "Adding a series resistor in the switch node limits the\npeak high-side driver current during turn-off, which\naffects the switching speed of the high-side driver. The\nresistor in series with the HO pin may be reduced to\nhelp compensate for the extra HS pin resistance."
- note added: "An external resistor between the\nLO output and the MOSFET may affect\nthe performance of the LO pin monitoring\ncircuit and is not recommended."
- moved on the sheet: C1, C10, C12, C13, C3, C4, C5, C7, C8, C9, D1, D2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
