File: board/SolarCurrentMonitor.sch (KiCad schematic (older format))
At the start: 3 parts, among them U3 INA260

Commit message: Rev 2 of board layout, WIP
Parts:
- C14, C15: footprint Capacitor_SMD:C_0805_2012Metric -> Capacitor_SMD:C_0805_2012Metric_Pad1.15x1.40mm_HandSolder
Changed lines of the file:
@@
 EESchema Schematic File Version 4
 LIBS:MPPTSolarCharger-cache
-EELAYER 26 0
+EELAYER 30 0
 EELAYER END
 $Descr A4 11693 8268
@@
 F 0 "C14" H 4115 3946 50  0000 L CNN
 F 1 "100nF" H 4115 3855 50  0000 L CNN
-F 2 "Capacitor_SMD:C_0805_2012Metric" H 4038 3750 50  0001 C CNN
+F 2 "Capacitor_SMD:C_0805_2012Metric_Pad1.15x1.40mm_HandSolder" H 4038 3750 50  0001 C CNN
 F 3 "~" H 4000 3900 50  0001 C CNN
 	1    4000 3900
@@
 F 0 "C15" H 5215 2996 50  0000 L CNN
 F 1 "100nF" H 5215 2905 50  0000 L CNN
-F 2 "Capacitor_SMD:C_0805_2012Metric" H 5138 2800 50  0001 C CNN
+F 2 "Capacitor_SMD:C_0805_2012Metric_Pad1.15x1.40mm_HandSolder" H 5138 2800 50  0001 C CNN
 F 3 "~" H 5100 2950 50  0001 C CNN
 	1    5100 2950
