File: board/BatteryCurrentMonitor.kicad_sch (KiCad schematic)
At the start: 3 parts

Commit message: Different board layout, WIP
Parts:
- C16, C17: renamed from C?; value (none) -> 100nF; footprint (none) -> Capacitor_SMD:C_0805_2012Metric_Pad1.18x1.45mm_HandSolder
- U4: renamed from U?; value (none) -> INA260; footprint (none) -> Package_SO:TSSOP-16_4.4x5mm_P0.65mm
Changed lines of the file:
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@@
   (symbol (lib_id "SaintGimp:INA260") (at 144.78 95.25 0) (unit 1)
     (in_bom yes) (on_board yes)
-    (property "Reference" "U?" (id 0) (at 139.7 83.82 0))
-    (property "Value" "" (id 1) (at 148.59 83.82 0))
-    (property "Footprint" "" (id 2) (at 144.78 109.22 0)
+    (property "Reference" "U4" (id 0) (at 139.7 83.82 0))
+    (property "Value" "INA260" (id 1) (at 148.59 83.82 0))
+    (property "Footprint" "Package_SO:TSSOP-16_4.4x5mm_P0.65mm" (id 2) (at 144.78 109.22 0)
       (effects (font (size 1.27 1.27)) hide)
     )
@@
   (symbol (lib_id "Device:C") (at 121.92 100.33 0) (unit 1)
     (in_bom yes) (on_board yes)
-    (property "Reference" "C?" (id 0) (at 124.841 99.1616 0)
+    (property "Reference" "C16" (id 0) (at 124.841 99.1616 0)
       (effects (font (size 1.27 1.27)) (justify left))
     )
-    (property "Value" "" (id 1) (at 124.841 101.473 0)
+    (property "Value" "100nF" (id 1) (at 124.841 101.473 0)
       (effects (font (size 1.27 1.27)) (justify left))
     )
-    (property "Footprint" "" (id 2) (at 122.8852 104.14 0)
+    (property "Footprint" "Capacitor_SMD:C_0805_2012Metric_Pad1.18x1.45mm_HandSolder" (id 2) (at 122.8852 104.14 0)
       (effects (font (size 1.27 1.27)) hide)
     )
@@
   (symbol (lib_id "power:GND") (at 121.92 105.41 0) (unit 1)
     (in_bom yes) (on_board yes)
-    (property "Reference" "#PWR?" (id 0) (at 121.92 111.76 0)
+    (property "Reference" "#PWR014" (id 0) (at 121.92 111.76 0)
       (effects (font (size 1.27 1.27)) hide)
     )
-    (property "Value" "" (id 1) (at 122.047 109.8042 0))
+    (property "Value" "GND" (id 1) (at 122.047 109.8042 0))
     (property "Footprint" "" (id 2) (at 121.92 105.41 0)
       (effects (font (size 1.27 1.27)) hide)
@@
   (symbol (lib_id "power:+3.3V") (at 144.78 67.31 0) (unit 1)
     (in_bom yes) (on_board yes)
-    (property "Reference" "#PWR?" (id 0) (at 144.78 71.12 0)
+    (property "Reference" "#PWR016" (id 0) (at 144.78 71.12 0)
       (effects (font (size 1.27 1.27)) hide)
     )
-    (property "Value" "" (id 1) (at 145.161 62.9158 0))
+    (property "Value" "+3.3V" (id 1) (at 145.161 62.9158 0))
     (property "Footprint" "" (id 2) (at 144.78 67.31 0)
       (effects (font (size 1.27 1.27)) hide)
@@
   (symbol (lib_id "power:GND") (at 144.78 107.95 0) (unit 1)
     (in_bom yes) (on_board yes)
-    (property "Reference" "#PWR?" (id 0) (at 144.78 114.3 0)
+    (property "Reference" "#PWR017" (id 0) (at 144.78 114.3 0)
       (effects (font (size 1.27 1.27)) hide)
     )
-    (property "Value" "" (id 1) (at 144.907 112.3442 0))
+    (property "Value" "GND" (id 1) (at 144.907 112.3442 0))
     (property "Footprint" "" (id 2) (at 144.78 107.95 0)
       (effects (font (size 1.27 1.27)) hide)
@@
   (symbol (lib_id "Device:C") (at 151.13 72.39 0) (unit 1)
     (in_bom yes) (on_board yes)
-    (property "Reference" "C?" (id 0) (at 154.051 71.2216 0)
+    (property "Reference" "C17" (id 0) (at 154.051 71.2216 0)
       (effects (font (size 1.27 1.27)) (justify left))
     )
-    (property "Value" "" (id 1) (at 154.051 73.533 0)
+    (property "Value" "100nF" (id 1) (at 154.051 73.533 0)
       (effects (font (size 1.27 1.27)) (justify left))
     )
-    (property "Footprint" "" (id 2) (at 152.0952 76.2 0)
+    (property "Footprint" "Capacitor_SMD:C_0805_2012Metric_Pad1.18x1.45mm_HandSolder" (id 2) (at 152.0952 76.2 0)
       (effects (font (size 1.27 1.27)) hide)
     )
@@
   (symbol (lib_id "power:GND") (at 151.13 76.2 0) (unit 1)
     (in_bom yes) (on_board yes)
-    (property "Reference" "#PWR?" (id 0) (at 151.13 82.55 0)
+    (property "Reference" "#PWR018" (id 0) (at 151.13 82.55 0)
       (effects (font (size 1.27 1.27)) hide)
     )
-    (property "Value" "" (id 1) (at 151.257 80.5942 0))
+    (property "Value" "GND" (id 1) (at 151.257 80.5942 0))
     (property "Footprint" "" (id 2) (at 151.13 76.2 0)
       (effects (font (size 1.27 1.27)) hide)
@@
   (symbol (lib_id "power:GND") (at 132.08 101.6 0) (unit 1)
     (in_bom yes) (on_board yes)
-    (property "Reference" "#PWR?" (id 0) (at 132.08 107.95 0)
+    (property "Reference" "#PWR015" (id 0) (at 132.08 107.95 0)
       (effects (font (size 1.27 1.27)) hide)
     )
-    (property "Value" "" (id 1) (at 132.207 105.9942 0))
+    (property "Value" "GND" (id 1) (at 132.207 105.9942 0))
     (property "Footprint" "" (id 2) (at 132.08 101.6 0)
       (effects (font (size 1.27 1.27)) hide)
