File: board/SolarCurrentMonitor.kicad_sch (KiCad schematic)
At the start: 3 parts

Commit message: Different board layout, WIP
Parts:
- C14, C15: renamed from C?; value (none) -> 100nF; footprint (none) -> Capacitor_SMD:C_0805_2012Metric_Pad1.18x1.45mm_HandSolder
- U3: renamed from U?; value (none) -> INA260; footprint (none) -> Package_SO:TSSOP-16_4.4x5mm_P0.65mm
Changed lines of the file:
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@@
   (symbol (lib_id "SaintGimp:INA260") (at 123.19 97.79 0) (unit 1)
     (in_bom yes) (on_board yes)
-    (property "Reference" "U?" (id 0) (at 118.11 86.36 0))
-    (property "Value" "" (id 1) (at 127 86.36 0))
-    (property "Footprint" "" (id 2) (at 123.19 111.76 0)
+    (property "Reference" "U3" (id 0) (at 118.11 86.36 0))
+    (property "Value" "INA260" (id 1) (at 127 86.36 0))
+    (property "Footprint" "Package_SO:TSSOP-16_4.4x5mm_P0.65mm" (id 2) (at 123.19 111.76 0)
       (effects (font (size 1.27 1.27)) hide)
     )
@@
   (symbol (lib_id "Device:C") (at 101.6 99.06 0) (unit 1)
     (in_bom yes) (on_board yes)
-    (property "Reference" "C?" (id 0) (at 104.521 97.8916 0)
+    (property "Reference" "C14" (id 0) (at 104.521 97.8916 0)
       (effects (font (size 1.27 1.27)) (justify left))
     )
-    (property "Value" "" (id 1) (at 104.521 100.203 0)
+    (property "Value" "100nF" (id 1) (at 104.521 100.203 0)
       (effects (font (size 1.27 1.27)) (justify left))
     )
-    (property "Footprint" "" (id 2) (at 102.5652 102.87 0)
+    (property "Footprint" "Capacitor_SMD:C_0805_2012Metric_Pad1.18x1.45mm_HandSolder" (id 2) (at 102.5652 102.87 0)
       (effects (font (size 1.27 1.27)) hide)
     )
@@
   (symbol (lib_id "power:GND") (at 101.6 105.41 0) (unit 1)
     (in_bom yes) (on_board yes)
-    (property "Reference" "#PWR?" (id 0) (at 101.6 111.76 0)
+    (property "Reference" "#PWR09" (id 0) (at 101.6 111.76 0)
       (effects (font (size 1.27 1.27)) hide)
     )
-    (property "Value" "" (id 1) (at 101.727 109.8042 0))
+    (property "Value" "GND" (id 1) (at 101.727 109.8042 0))
     (property "Footprint" "" (id 2) (at 101.6 105.41 0)
       (effects (font (size 1.27 1.27)) hide)
@@
   (symbol (lib_id "power:+3.3V") (at 123.19 69.85 0) (unit 1)
     (in_bom yes) (on_board yes)
-    (property "Reference" "#PWR?" (id 0) (at 123.19 73.66 0)
+    (property "Reference" "#PWR011" (id 0) (at 123.19 73.66 0)
       (effects (font (size 1.27 1.27)) hide)
     )
-    (property "Value" "" (id 1) (at 123.571 65.4558 0))
+    (property "Value" "+3.3V" (id 1) (at 123.571 65.4558 0))
     (property "Footprint" "" (id 2) (at 123.19 69.85 0)
       (effects (font (size 1.27 1.27)) hide)
@@
   (symbol (lib_id "power:GND") (at 123.19 110.49 0) (unit 1)
     (in_bom yes) (on_board yes)
-    (property "Reference" "#PWR?" (id 0) (at 123.19 116.84 0)
+    (property "Reference" "#PWR012" (id 0) (at 123.19 116.84 0)
       (effects (font (size 1.27 1.27)) hide)
     )
-    (property "Value" "" (id 1) (at 123.317 114.8842 0))
+    (property "Value" "GND" (id 1) (at 123.317 114.8842 0))
     (property "Footprint" "" (id 2) (at 123.19 110.49 0)
       (effects (font (size 1.27 1.27)) hide)
@@
   (symbol (lib_id "power:GND") (at 110.49 105.41 0) (unit 1)
     (in_bom yes) (on_board yes)
-    (property "Reference" "#PWR?" (id 0) (at 110.49 111.76 0)
+    (property "Reference" "#PWR010" (id 0) (at 110.49 111.76 0)
       (effects (font (size 1.27 1.27)) hide)
     )
-    (property "Value" "" (id 1) (at 110.617 109.8042 0))
+    (property "Value" "GND" (id 1) (at 110.617 109.8042 0))
     (property "Footprint" "" (id 2) (at 110.49 105.41 0)
       (effects (font (size 1.27 1.27)) hide)
@@
   (symbol (lib_id "Device:C") (at 129.54 74.93 0) (unit 1)
     (in_bom yes) (on_board yes)
-    (property "Reference" "C?" (id 0) (at 132.461 73.7616 0)
+    (property "Reference" "C15" (id 0) (at 132.461 73.7616 0)
       (effects (font (size 1.27 1.27)) (justify left))
     )
-    (property "Value" "" (id 1) (at 132.461 76.073 0)
+    (property "Value" "100nF" (id 1) (at 132.461 76.073 0)
       (effects (font (size 1.27 1.27)) (justify left))
     )
-    (property "Footprint" "" (id 2) (at 130.5052 78.74 0)
+    (property "Footprint" "Capacitor_SMD:C_0805_2012Metric_Pad1.18x1.45mm_HandSolder" (id 2) (at 130.5052 78.74 0)
       (effects (font (size 1.27 1.27)) hide)
     )
@@
   (symbol (lib_id "power:GND") (at 129.54 78.74 0) (unit 1)
     (in_bom yes) (on_board yes)
-    (property "Reference" "#PWR?" (id 0) (at 129.54 85.09 0)
+    (property "Reference" "#PWR013" (id 0) (at 129.54 85.09 0)
       (effects (font (size 1.27 1.27)) hide)
     )
-    (property "Value" "" (id 1) (at 129.667 83.1342 0))
+    (property "Value" "GND" (id 1) (at 129.667 83.1342 0))
     (property "Footprint" "" (id 2) (at 129.54 78.74 0)
       (effects (font (size 1.27 1.27)) hide)
